File: RaspiBBHat.kicad_pcb (KiCad board)
At the start: 2 copper layers, 56.6 x 65.5 mm, 9 parts, among them J1 Conn_01x03, J2 Conn_01x16, J3 Conn_01x03, J4 Conn_01x16, J5 Raspberry_Pi_2_3

Commit message: Apply larger clearance mounting holes
Parts:
- REF1, REF2, REF3, REF4: footprint MountingHole:MountingHole_2.7mm -> Footprints:LargeClearanceMountingHole_2.7mm
Changed lines of the file:
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@@
     (add_net ID_SD)
   )
-  (module MountingHole:MountingHole_2.7mm (layer F.Cu)
+  (module Footprints:LargeClearanceMountingHole_2.7mm (layer F.Cu)
     (at 76.095 71.33)
     (descr "Mounting Hole 2.7mm, no annular")
@@
     (fp_circle (center 0 0) (end 2.95 0) (layer F.CrtYd) (width 0.05))
     (fp_circle (center 0 0) (end 2.7 0) (layer Cmts.User) (width 0.15))
-    (fp_text user %R (at 0.343 -0.007) (layer F.Fab)
-      (effects (font (size 1 1) (thickness 0.15)))
-    )
-    (pad 1 np_thru_hole circle (at 0 0) (size 2.7 2.7) (drill 2.7) (layers *.Cu *.Mask))
+    (fp_text user %R (at 0.3 0) (layer F.Fab)
+      (effects (font (size 1 1) (thickness 0.15)))
+    )
+    (pad "" np_thru_hole circle (at 0 0) (size 2.7 2.7) (drill 2.7) (layers *.Cu *.Mask)
+      (solder_mask_margin 1.3) (clearance 1.6))
+  )
+  (module Footprints:LargeClearanceMountingHole_2.7mm (layer F.Cu)
+    (at 76.095 129.33)
+    (descr "Mounting Hole 2.7mm, no annular")
+    (tags "mounting hole 2.7mm no annular")
+    (attr virtual)
+    (fp_text reference REF4 (at 0 -3.7) (layer F.SilkS) hide
+      (effects (font (size 1 1) (thickness 0.15)))
+    )
+    (fp_text value MountingHole_2.7mm (at 0 3.7) (layer F.Fab) hide
+      (effects (font (size 1 1) (thickness 0.15)))
+    )
+    (fp_circle (center 0 0) (end 2.95 0) (layer F.CrtYd) (width 0.05))
+    (fp_circle (center 0 0) (end 2.7 0) (layer Cmts.User) (width 0.15))
+    (fp_text user %R (at 0.3 0) (layer F.Fab)
+      (effects (font (size 1 1) (thickness 0.15)))
+    )
+    (pad "" np_thru_hole circle (at 0 0) (size 2.7 2.7) (drill 2.7) (layers *.Cu *.Mask)
+      (solder_mask_margin 1.3) (clearance 1.6))
+  )
+  (module Footprints:LargeClearanceMountingHole_2.7mm (layer F.Cu)
+    (at 125.095 129.33)
+    (descr "Mounting Hole 2.7mm, no annular")
+    (tags "mounting hole 2.7mm no annular")
+    (attr virtual)
+    (fp_text reference REF3 (at 0 -3.7) (layer F.SilkS) hide
+      (effects (font (size 1 1) (thickness 0.15)))
+    )
+    (fp_text value MountingHole_2.7mm (at 0 3.7) (layer F.Fab) hide
+      (effects (font (size 1 1) (thickness 0.15)))
+    )
+    (fp_circle (center 0 0) (end 2.95 0) (layer F.CrtYd) (width 0.05))
+    (fp_circle (center 0 0) (end 2.7 0) (layer Cmts.User) (width 0.15))
+    (fp_text user %R (at 0.3 0) (layer F.Fab)
+      (effects (font (size 1 1) (thickness 0.15)))
+    )
+    (pad "" np_thru_hole circle (at 0 0) (size 2.7 2.7) (drill 2.7) (layers *.Cu *.Mask)
+      (solder_mask_margin 1.3) (clearance 1.6))
+  )
+  (module Footprints:LargeClearanceMountingHole_2.7mm (layer F.Cu)
+    (at 125.095 71.33)
+    (descr "Mounting Hole 2.7mm, no annular")
+    (tags "mounting hole 2.7mm no annular")
+    (attr virtual)
+    (fp_text reference REF2 (at 0 -3.7) (layer F.SilkS) hide
+      (effects (font (size 1 1) (thickness 0.15)))
+    )
+    (fp_text value MountingHole_2.7mm (at 0 3.7) (layer F.Fab) hide
+      (effects (font (size 1 1) (thickness 0.15)))
+    )
+    (fp_circle (center 0 0) (end 2.95 0) (layer F.CrtYd) (width 0.05))
+    (fp_circle (center 0 0) (end 2.7 0) (layer Cmts.User) (width 0.15))
+    (fp_text user %R (at 0.3 0) (layer F.Fab)
+      (effects (font (size 1 1) (thickness 0.15)))
+    )
+    (pad "" np_thru_hole circle (at 0 0) (size 2.7 2.7) (drill 2.7) (layers *.Cu *.Mask)
+      (solder_mask_margin 1.3) (clearance 1.6))
   )
   (module Connector_PinSocket_2.54mm:PinSocket_1x03_P2.54mm_Vertical (layer F.Cu)
@@
     )
   )
-  (module MountingHole:MountingHole_2.7mm (layer F.Cu)
-    (at 125.095 71.33)
-    (descr "Mounting Hole 2.7mm, no annular")
-    (tags "mounting hole 2.7mm no annular")
-    (attr virtual)
-    (fp_text reference REF2 (at 0 -3.7) (layer F.SilkS) hide
-      (effects (font (size 1 1) (thickness 0.15)))
-    )
-    (fp_text value MountingHole_2.7mm (at 0 3.7) (layer F.Fab) hide
-      (effects (font (size 1 1) (thickness 0.15)))
-    )
-    (fp_circle (center 0 0) (end 2.95 0) (layer F.CrtYd) (width 0.05))
-    (fp_circle (center 0 0) (end 2.7 0) (layer Cmts.User) (width 0.15))
-    (fp_text user %R (at 0.3 0) (layer F.Fab)
-      (effects (font (size 1 1) (thickness 0.15)))
-    )
-    (pad 1 np_thru_hole circle (at 0 0) (size 2.7 2.7) (drill 2.7) (layers *.Cu *.Mask))
-  )
-  (module MountingHole:MountingHole_2.7mm (layer F.Cu)
-    (at 76.095 129.33)
-    (descr "Mounting Hole 2.7mm, no annular")
-    (tags "mounting hole 2.7mm no annular")
-    (attr virtual)
-    (fp_text reference REF4 (at 0 -3.7) (layer F.SilkS) hide
-      (effects (font (size 1 1) (thickness 0.15)))
-    )
-    (fp_text value MountingHole_2.7mm (at 0 3.7) (layer F.Fab) hide
-      (effects (font (size 1 1) (thickness 0.15)))
-    )
-    (fp_circle (center 0 0) (end 2.95 0) (layer F.CrtYd) (width 0.05))
-    (fp_circle (center 0 0) (end 2.7 0) (layer Cmts.User) (width 0.15))
-    (fp_text user %R (at 0.3 0) (layer F.Fab)
-      (effects (font (size 1 1) (thickness 0.15)))
-    )
-    (pad 1 np_thru_hole circle (at 0 0) (size 2.7 2.7) (drill 2.7) (layers *.Cu *.Mask))
-  )
-  (module MountingHole:MountingHole_2.7mm (layer F.Cu)
-    (at 125.095 129.33)
-    (descr "Mounting Hole 2.7mm, no annular")
-    (tags "mounting hole 2.7mm no annular")
-    (attr virtual)
-    (fp_text reference REF3 (at 0 -3.7) (layer F.SilkS) hide
-      (effects (font (size 1 1) (thickness 0.15)))
-    )
-    (fp_text value MountingHole_2.7mm (at 0 3.7) (layer F.Fab) hide
-      (effects (font (size 1 1) (thickness 0.15)))
-    )
-    (fp_circle (center 0 0) (end 2.95 0) (layer F.CrtYd) (width 0.05))
-    (fp_circle (center 0 0) (end 2.7 0) (layer Cmts.User) (width 0.15))
-    (fp_text user %R (at 0.3 0) (layer F.Fab)
-      (effects (font (size 1 1) (thickness 0.15)))
-    )
-    (pad 1 np_thru_hole circle (at 0 0) (size 2.7 2.7) (drill 2.7) (layers *.Cu *.Mask))
-  )
   (gr_text "github.com/asukiaaa/RaspiBBHat\n" (at 73.5965 99.822 270) (layer B.SilkS)
